File: SURF.kicad_sch (KiCad schematic)
At the start: 78 parts, among them Q1 BC338, Q2 BC338, Q3 Q_Dual_PMOS_S1G1D2S2G2D1, Q4 BC338, SW1 SW_MEC_5E, SW3 SW_MEC_5E, U1 ESP32-S2-MINI-2, U10 COMM_10_RIGHT, U11 CONN_10_LEFT, U2 CP2102N-A02-GQFN28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

Commit message: update
Parts:
- removed C11, C13: 10uF/25V(20%), symbol Device:C
- removed C12, C14: 0.1uF/50V(10%), symbol Device:C
- removed U4: SGM2212, symbol New_2:SGM2212
- D1: value RED LED -> LED
- R18: value 5.1K(1%) -> 1K
- U5: footprint (none) -> new:1051640001
Connections:
- net +3.3V: now also R18.2
- net GND: no longer D1.1 (K)
- net GPIO18: no longer R17.1
- net GPIO21: now also R17.1
- net GPIO33: now also D1.1 (K)
- net at R18.1: now also D1.2 (A)
- net VBUS: now reaches 22.1K(1%)1.2, D4.1 (A1), D7.2 (A), U5.1 (VBUS)
- no-connect marks 56 -> 55
Other:
- moved on the sheet: Q4, R25, R26, U9

Commit message: new
Parts:
- removed 22.1K(1%)1: R, symbol Device:R
- removed C10, C7: 22pF/50V(5%)(NC), symbol Device:C
- removed C23, C24: 0.1uF/50V(10%)(NC), symbol Device:C
- removed C8: 10uF/25V(20%), symbol Device:C
- removed C9: 1uF/16V/(10%), symbol Device:C
- removed D4, D5, D6: 1.5KExxCA, Diode_THT:D_DO-201AE_P15.24mm_Horizontal, symbol Diode:1.5KExxCA
- removed D7: 1N914, Diode_THT:D_DO-35_SOD27_P7.62mm_Horizontal, symbol Diode:1N914
- removed Q1, Q2: BC338, Package_TO_SOT_THT:TO-92_Inline, symbol Transistor_BJT:BC338
- removed R10: 47.5K(1%), symbol Device:R
- removed R11, R12: 0(1%)(NC), symbol Device:R
- removed R13, R6, R7: 0(1%), symbol Device:R
- removed R14, R15, R16, R17, R4, R5: 10K(1%), symbol Device:R
- removed R8: 10K(1%)(NC), symbol Device:R
- removed R9: 1K(1%), symbol Device:R
- removed SW1, SW3: SW_MEC_5E, symbol Switch:SW_MEC_5E
- removed U2: CP2102N-A02-GQFN28, CP2102N-A02-GQFN28:QFN50P500X500X80-29N, symbol CP2102N:CP2102N-A02-GQFN28
- removed U3: SK68XXMINI-HS, SK6812MINI:SK6812MINI, symbol New:SK68XXMINI
- removed U5: MICRO USB, new:1051640001, symbol New_2:Micro_USB
- added J1, J2: Conn_01x21_Pin, symbol Connector:Conn_01x21_Pin
- added SW1, SW2: SW_Omron_B3FS, symbol Switch:SW_Omron_B3FS
- added U2: UART, symbol New:UART
- C3: value 22pF/50V(5%)(NC) -> TBD
- C6: value 10uF/25V(20%) -> 0.1uF
- R2: value 0(1%) -> TBD
- R3: value 0(1%) -> 0
- U1: footprint (none) -> new:ESP32-S2-MINI-2
Connections:
- net CHIP_PU is gone; now on an unnamed net: U1.45 (EN)
- net +3.3V: no longer C6.1
- net GND: now also C3.1, SW1.1, SW2.1, U2.4; no longer C3.2
- net GPIO0: now also SW1.2
- net GPIO1: no longer R24.2
- net GPIO17: now also U10.2 (E_RX2); no longer U10.1 (E_TX2)
- net GPIO18: now also U10.1 (E_TX2); no longer U10.2 (E_RX2)
- net at U1.24 (IO20): no longer C3.1
- net EN: now reaches R3.1
- net at U1.39 (TXD0): now also U2.3; no longer R3.2
- net VDD: now reaches R2.1
- net VDD: now also U2.1
- net at R2.2: now also C3.2; no longer U1.40 (RXD0)
- new net: U1.40 (RXD0), U2.2
- new net: C6.1, R3.2, SW2.2
- new net GPIO1(CAM_PWR): R24.2
- no-connect marks 55 -> 35
Other:
- note added: "VDD33"
- note removed: "RBG_CTRL"
- moved on the sheet: +C18, C1, C15, C16, C17, C18, C19, C2, C20, C21, C22, C25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

Commit message: new
Parts:
- removed C25: 0.1uF, symbol Device:C
- removed Q4: BC338, Package_TO_SOT_THT:TO-92_Inline, symbol Transistor_BJT:BC338
- removed R22: 4.7K, symbol Device:R
- removed R25: 10K, symbol Device:R
- removed R26: 1K, symbol Device:R
- removed U9: LED_FLASH, symbol New_2:LED_FLASH
Connections:
- net +3V0: now also J1.1 (Pin_1), J1.20 (Pin_20)
- net EN: now also J2.2 (Pin_2)
- net GND: now also J1.21 (Pin_21), J2.1 (Pin_1)
- net GPIO0: now also J1.2 (Pin_2)
- net GPIO1: now also J1.3 (Pin_3)
- net GPIO10: now also J1.12 (Pin_12)
- net GPIO11: now also J1.13 (Pin_13)
- net GPIO12: now also J1.14 (Pin_14)
- net GPIO13: now also J1.15 (Pin_15)
- net GPIO14: now also J1.16 (Pin_16)
- net GPIO15: now also J1.17 (Pin_17)
- net GPIO16: now also J1.18 (Pin_18)
- net GPIO17: now also J1.19 (Pin_19)
- net GPIO18: now also J2.21 (Pin_21)
- net GPIO2: now also J1.4 (Pin_4)
- net GPIO21: now also J2.18 (Pin_18)
- net GPIO26: now also J2.17 (Pin_17)
- net GPIO3: now also J1.5 (Pin_5)
- net GPIO33: now also J2.16 (Pin_16)
- net GPIO34: now also J2.15 (Pin_15)
- net GPIO35: now also J2.14 (Pin_14)
- net GPIO36: now also J2.13 (Pin_13)
- net GPIO37: now also J2.12 (Pin_12)
- net GPIO38: now also J2.11 (Pin_11)
- net GPIO39: now also J2.10 (Pin_10)
- net GPIO4: now also J1.6 (Pin_6)
- net GPIO40: now also J2.9 (Pin_9)
- net GPIO41: now also J2.8 (Pin_8)
- net GPIO42: now also J2.7 (Pin_7)
- net GPIO45: now also J2.4 (Pin_4)
- net GPIO46: now also J2.3 (Pin_3)
- net GPIO5: now also J1.7 (Pin_7)
- net GPIO6: now also J1.8 (Pin_8)
- net GPIO7: now also J1.9 (Pin_9)
- net GPIO8: now also J1.10 (Pin_10)
- net GPIO9: now also J1.11 (Pin_11)
- net GPIO20: now reaches J2.19 (Pin_19)
- net GPIO19: now reaches J2.20 (Pin_20)
- net U0RXD: now reaches J2.5 (Pin_5)
- net U0TXD: now reaches J2.6 (Pin_6)
Other:
- note added: "VCC_3V3"
- note added: "VCC_5V"
- moved on the sheet: J1, J2

Commit message: update
Parts:
- removed R2: TBD, symbol Device:R
- removed U7, U8: XC6206PxxxMR, Package_TO_SOT_SMD:SOT-23-3, symbol Regulator_Linear:XC6206PxxxMR
- added IC1: TPS7A0212PDBVR, SOT95P280X145-5N, symbol TPS7A0212PDBVR:TPS7A0212PDBVR
- added IC2: TPS7A0228PDBVR, SOT95P280X145-5N, symbol TPS7A0228PDBVR:TPS7A0228PDBVR
- added R4: 499 ohms, symbol Device:R
- C3: value TBD -> 10uF
- SW1, SW2: footprint (none) -> B3FS:B3FS1012
Connections:
- net +1V2: now also IC1.5 (OUT)
- net +2V8: now also IC2.5 (OUT)
- net GND: now also IC1.2 (GND), IC2.2 (GND)
- net GPIO13: now also D1.1 (K)
- net GPIO17: now also U2.3; no longer U10.2 (E_RX2)
- net GPIO18: now also U2.2; no longer U10.1 (E_TX2)
- net GPIO33: no longer D1.1 (K)
- net at C18.1, Q3.1 (S): now also IC1.1 (IN), IC2.1 (IN)
- net E_TX2: now reaches U1.40 (RXD0)
- net E_TX2: no longer U2.2
- net at U1.39 (TXD0): now also R4.2; no longer U2.3
- new net E_RX2: R4.1
- new net RXD0: U10.1 (E_TX2)
- new net TXD0: U10.2 (E_RX2)
- no-connect marks 35 -> 38
Other:
- moved on the sheet: C19, C20, C21, C3, C4, C5, C6, D1, R18, R27, R28, R3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

Commit message: new update
Parts:
- added R2: 0, symbol Device:R
- R4: value 499 ohms -> 499 ohms R
Connections:
- net +3.3V is gone; now on net +3V3: C4.1, C5.1, R18.2, U1.3 (3V3)
- net E_TX2 is gone; now on net RXD0: U1.40 (RXD0)
- net GPIO1(CAM_PWR) is gone; now on net GPIO1: R24.2
- net U0RXD is gone; now on net RXD0: J2.5 (Pin_5)
- net U0TXD is gone; now on net TXD0: J2.6 (Pin_6)
- net VDD is gone; now on net +3V3: U2.1
- net +3V0: no longer J1.1 (Pin_1), J1.20 (Pin_20)
- net +3V3: now also J1.1 (Pin_1), R2.1
- net +5V: now also J1.20 (Pin_20)
- net EN: now also C3.2, U1.45 (EN), R2.2
- net E_RX2: now also U10.2 (E_RX2)
- net GPIO19: now also U1.23 (IO19)
- net GPIO20: now also U1.24 (IO20)
- net TXD0: now also R4.2, U1.39 (TXD0); no longer U10.2 (E_RX2)
- net SW_EN: now reaches C6.1, R3.2, SW2.2
- no-connect marks 38 -> 37
Other:
- note added: "(CAM_PWR)"
- moved on the sheet: R3, R4, SW1

Commit message: new update
Parts:
- removed U2: UART, symbol New:UART
- added J3: Conn_01x04, symbol Connector_Generic:Conn_01x04
Connections:
- net +3V3: now also J3.1 (Pin_1)
- net GND: now also J3.4 (Pin_4)
- net GPIO17: now also J3.2 (Pin_2)
- net GPIO18: now also J3.3 (Pin_3)
Other:
- note added: "BOOT SWITCH"
- note added: "CrazyFlie Connectors"
- note added: "ESP32-S2-MINI-2 MODULE"
- note added: "LED AND POWER SUPPLY"
- note added: "OV2640 CAM MODULE"
- note added: "Pin Headers for ESP32-S2-MINI-2"
- note added: "Power Flags"
- note added: "Power Supply for CAM_RST"
- note added: "Power Supply for OV2640"
- note added: "Power Supply for SCK and SDA"
- note added: "RESET SWITCH"
- note added: "SURF Vision Offloading Module"
- note added: "UART"
- moved on the sheet: +C18, C1, C15, C16, C17, C18, C19, C2, C20, C21, C22, C3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

Commit message: new update
Other:
- note removed: "SURF Vision Offloading Module"
- company: (none) -> Effecient Computing Lab
- title: (none) -> SURF Vision Offloading Module
Changed lines of the file:
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@@
 (kicad_sch (version 20230121) (generator eeschema)
   (paper "A4")
+  (title_block
+    (title "SURF Vision Offloading Module")
+    (date "2023-07-07")
+    (company "Effecient Computing Lab")
+    (comment 1 "Put together by Kimberly By Goytia")
+  )
   (junction (at 48.26 60.96) (diameter 0) (color 0 0 0 0)
   )
@@
     (effects (font (size 1.27 1.27)) (justify left bottom))
   )
-  (text "SURF Vision Offloading Module" (at 186.69 190.5 0)
-    (effects (font (size 1.5 1.5) (thickness 0.3) bold) (justify left bottom))
-  )
   (text "RESET SWITCH" (at 255.27 39.37 0)

Commit message: new update
Parts:
- removed J3: Conn_01x04, symbol Connector_Generic:Conn_01x04
- removed R2: 0, symbol Device:R
- +C18: footprint LED_SMD:LED_SK6812MINI_PLCC4_3.5x3.5mm_P1.75mm -> CAPACITOR100UF:CAPC2012X135N
- C1: footprint (none) -> CAPACITOR15PF:CAPC1608X87N
- C15, C2, C20, C21, C6: footprint (none) -> CAPACITOR0.1UF:CAPC1608X90N
- C16, C17, C18, C19, C22, C3: footprint (none) -> CAPACITOR10UF:CAPC2012X145N
- C4, C5: footprint (none) -> CAPACITOR0.1UF50V:CAPC3216X170N
- D1: footprint (none) -> LED_SMD:LED_0603_1608Metric
- IC1: footprint SOT95P280X145-5N -> TPS7A0212PDBVR:SOT95P280X145-5N
- IC2: footprint SOT95P280X145-5N -> TPS7A0228PDBVR:SOT95P280X145-5N
- J1, J2: footprint (none) -> Connector_PinHeader_2.54mm:PinHeader_1x21_P2.54mm_Vertical
- Q3: footprint (none) -> Package_TO_SOT_SMD:SOT-363_SC-70-6
- R1, R18, R19, R20, R21, R23, R24, R27, R28, R3: footprint (none) -> Resistor_SMD:R_0402_1005Metric
- R4: value 499 ohms R -> 499 R; footprint (none) -> Resistor_SMD:R_0402_1005Metric
- U6: footprint KiCad:SOT95P275X110-5N -> NCP164CSN300T1G:SOT95P275X110-5N
Other:
- note added: "POWER SUPPLY FOR LED"
- note removed: "LED AND POWER SUPPLY"
- note removed: "UART"
- note removed: "VDD33"
- moved on the sheet: C6, D1, R18, R3, SW2
