File: SURF.kicad_sch (KiCad schematic)
At the start: 39 parts, among them IC1 TPS7A0212PDBVR, IC2 TPS7A0228PDBVR, J1 Conn_01x21_Pin, J2 Conn_01x21_Pin, Q3 Q_Dual_PMOS_S1G1D2S2G2D1, SW1 SW_Omron_B3FS, SW2 SW_Omron_B3FS, U1 ESP32-S2-MINI-2, U10 COMM_10_RIGHT, U11 CONN_10_LEFT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

Commit message: new update
Parts:
- added C7, C8: 12pF, CAPACITOR12pF:CAPC0603X33N, symbol Device:C
- added R2, R5, R6: 0 NC, Resistor_SMD:R_0402_1005Metric, symbol Device:R
- added XTAL1: 32.768kHz (NC), CRYSTAL32.768kHz:ABS0532768KHZ7T, symbol dk_Crystals:ECS-_327-12_5-34B-TR
- R18: value 1K -> 5.1K
Connections:
- net GND: now also D1.1 (K), C7.2, C8.2
- net GPIO13: no longer D1.1 (K)
- net GPIO15: now also R5.1
- net GPIO16: now also R6.1
- new net: C8.1, R2.1, R6.2, XTAL1.1
- new net: C7.1, R2.2, R5.2, XTAL1.2
- no-connect marks 37 -> 35
Other:
- note added: "ANTENNA"
- moved on the sheet: +C18, C16, C17, C18, C19, C20, C21, C22, C6, D1, IC1, IC2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

Commit message: new update
Parts:
- removed +C18: 100uF, CAPACITOR100UF:CAPC2012X135N, symbol Device:C
- removed C16: 10uF, CAPACITOR10UF:CAPC2012X145N, symbol Device:C
- removed C7, C8: 12pF, CAPACITOR12pF:CAPC0603X33N, symbol Device:C
- removed J1, J2: Conn_01x21_Pin, Connector_PinHeader_2.54mm:PinHeader_1x21_P2.54mm_Vertical, symbol Connector:Conn_01x21_Pin
- removed R2, R5, R6: 0 NC, Resistor_SMD:R_0402_1005Metric, symbol Device:R
- removed R27, R28: 2.2K, Resistor_SMD:R_0402_1005Metric, symbol Device:R
- removed SW1, SW2: SW_Omron_B3FS, B3FS:B3FS1012, symbol Switch:SW_Omron_B3FS
- removed U10: COMM_10_RIGHT, symbol New_2:CONN_10_RIGHT
- removed U11: CONN_10_LEFT, symbol New_2:CONN_10_LEFT
- removed U6: NCP164CSN300T1G, NCP164CSN300T1G:SOT95P275X110-5N, symbol Regulator_Linear:AMS1117
- removed XTAL1: 32.768kHz (NC), CRYSTAL32.768kHz:ABS0532768KHZ7T, symbol dk_Crystals:ECS-_327-12_5-34B-TR
- added BOOT, RESET: TS20-42-25-WT-160-SMT-TR, NEW-SWITCH:TS204225WT160SMTTR, symbol TS20-42-25-WT-160-SMT-TR:TS20-42-25-WT-160-SMT-TR
- added J1: Conn_01x10_Pin RIGHT, CONN_01X10_CRAZTFLIE:CONN_PINHEADERS_01X10_CRAZYFLIE, symbol Connector:Conn_01x10_Pin
- added J2: Conn_01x10_Pin LEFT, CONN_01X10_CRAZTFLIE:CONN_PINHEADERS_01X10_CRAZYFLIE, symbol Connector:Conn_01x10_Pin
- added J3: Conn_01x04, Connector_PinHeader_2.54mm:PinHeader_1x04_P2.54mm_Vertical, symbol Connector_Generic:Conn_01x04
Connections:
- net +3V0: now also R18.2, R19.2, R20.2, R21.2, J3.1 (Pin_1); no longer C17.1, Q3.6 (D), R23.1
- net +3V3: no longer R18.2, R19.2, R20.2, R21.2
- net GND: now also BOOT.3 (COM_1), J2.10 (Pin_10), J3.4 (Pin_4), RESET.3 (COM_1)
- net GPIO0: now also BOOT.2 (NO_2)
- net GPIO17: now also J1.2 (Pin_2)
- net GPIO18: now also J1.1 (Pin_1)
- net RXD0: now also J3.2 (Pin_2)
- net SW_EN: now also RESET.2 (NO_2)
- net PWR_LED: now reaches D1.2 (A), R18.1
- net CAM_RST: no longer names the net of C15.2, CAM1.19 (RESET), R19.1
- net E_RX2: no longer names the net of R4.1
- net E_RX2: now also J3.3 (Pin_3)
- net TWI_SCK: no longer names the net of CAM1.20 (SIO_C), R20.1
- net TWI_SDA: no longer names the net of CAM1.22 (SIO_D), R21.1
- new net VCC: C17.1, J2.1 (Pin_1), Q3.6 (D), R23.1
- no-connect marks 35 -> 44
Other:
- note added: "UART PINS"
- note removed: "ANTENNA"
- note removed: "Pin Headers for ESP32-S2-MINI-2"
- note removed: "VCC_3V3"
- note removed: "VCC_5V"
- moved on the sheet: C17, C18, C19, C20, C21, C22, C6, D1, IC1, IC2, Q3A, R18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

Commit message: new update
Parts:
- added R2: 0, Resistor_SMD:R_0402_1005Metric, symbol Device:R
- renumbered BOOT to BOOT1, RESET to RESET1
Connections:
- net GPIO14 is gone; now on net TWI_SDA: U1.18 (IO14)
- net GPIO15 is gone; now on net TWI_SCK: U1.19 (IO15)
- net +3V0: now also C3.1, C4.1, C5.1, U1.3 (3V3)
- net GND: now also R2.2; no longer C3.1, RESET1.3 (COM_1)
- net GPIO10: now also CAM1.12 (XVCLK); no longer CAM1.13 (Y9)
- net GPIO11: now also CAM1.13 (Y9); no longer CAM1.16 (HREF)
- net GPIO12: now also CAM1.16 (HREF); no longer CAM1.18 (VSYNC)
- net GPIO13: now also CAM1.18 (VSYNC)
- net GPIO7: now also C1.1, CAM1.8 (PCLK); no longer CAM1.9 (Y7)
- net GPIO8: now also CAM1.9 (Y7); no longer CAM1.11 (Y8)
- net GPIO9: now also CAM1.11 (Y8); no longer CAM1.12 (XVCLK)
- net VCC: now also C2.1, CAM1.14 (DOVDD); no longer R23.1
- net TWI_SCK: now reaches CAM1.20 (SIO_C), R20.1
- net Y0: now reaches CAM1.1 (YO)
- net PWDN: now reaches CAM1.17 (PWDN), R1.1
- net RESET: now reaches C15.2, CAM1.19 (RESET), R19.1
- net Y1: now reaches CAM1.2 (Y1)
- net TWI_SDA: now reaches CAM1.22 (SIO_D), R21.1
- net at R23.2, R24.1: no longer Q3.2 (G)
- net at C18.1, IC1.1 (IN), IC2.1 (IN)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: now also R23.1
- removed net +3V3: C2.1, C4.1, C5.1, CAM1.14 (DOVDD), U1.3 (3V3)
- new net: R2.1, RESET1.3 (COM_1)
- no-connect marks 44 -> 42
Other:
- moved on the sheet: C6, J1, J2, Q3A, R23, R24

Commit message: new update
Parts:
- removed C3: 10uF, CAPACITOR10UF:CAPC2012X145N, symbol Device:C
- removed C6: 0.1uF, CAPACITOR0.1UF:CAPC1608X90N, symbol Device:C
- removed R2, R3: 0, Resistor_SMD:R_0402_1005Metric, symbol Device:R
- removed R23: 10K, Resistor_SMD:R_0402_1005Metric, symbol Device:R
- added R5: 10K, Resistor_SMD:R_0402_1005Metric, symbol Device:R
Connections:
- net EN is gone; now on net GND: U1.45 (EN)
- net SW_EN is gone; now on net GND: RESET1.2 (NO_2)
- net +3V0: now also R5.2
- net GND: now also RESET1.3 (COM_1), R5.1
- net VCC: no longer C2.1, CAM1.14 (DOVDD)
- net at R24.1: now also Q3.2 (G)
- net CAM_VCC: now reaches C18.1, IC1.1 (IN), IC2.1 (IN), Q3.1 (S)
- net CAM_VCC: now also C2.1, CAM1.14 (DOVDD), IC1.3 (EN), IC2.3 (EN)
- no-connect marks 42 -> 39
Other:
- moved on the sheet: C18, Q3A, R24

Commit message: new update
Connections:
- net GPIO16 is gone; now on net TWI_SCK: U1.20 (IO16)
- net GND: no longer R5.1, RESET1.2 (NO_2), U1.45 (EN)
- net TWI_SCK: no longer U1.19 (IO15)
- net TWI_SDA: now also U1.19 (IO15); no longer U1.18 (IO14)
- net RESET renamed GPIO14
- net GPIO14: now also U1.18 (IO14)
- new net EN: R5.1, RESET1.2 (NO_2), U1.45 (EN)
- no-connect marks 39 -> 38
Changed lines of the file:
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@@
   (junction (at 135.89 33.02) (diameter 0) (color 0 0 0 0)
   )
-  (junction (at 214.63 87.63) (diameter 0) (color 0 0 0 0)
-  )
   (junction (at 114.3 62.23) (diameter 0) (color 0 0 0 0)
   )
@@
   )
   (junction (at 60.96 83.82) (diameter 0) (color 0 0 0 0)
-  )
-  (junction (at 251.46 78.74) (diameter 0) (color 0 0 0 0)
   )
   (junction (at 167.64 20.32) (diameter 0) (color 0 0 0 0)
@@
   (no_connect (at 185.42 92.71))
   (no_connect (at 204.47 60.96))
-  (no_connect (at 165.1 92.71))
   (no_connect (at 187.96 142.24))
   (no_connect (at 204.47 55.88))
@@
     (stroke (width 0) (type default))
   )
-  (wire (pts (xy 251.46 78.74) (xy 251.46 87.63))
-    (stroke (width 0) (type default))
-  )
   (wire (pts (xy 190.5 20.32) (xy 190.5 25.4))
     (stroke (width 0) (type default))
@@
     (stroke (width 0) (type default))
   )
-  (wire (pts (xy 214.63 81.28) (xy 214.63 87.63))
-    (stroke (width 0) (type default))
-  )
   (wire (pts (xy 180.34 20.32) (xy 180.34 25.4))
     (stroke (width 0) (type default))
@@
     (stroke (width 0) (type default))
   )
+  (wire (pts (xy 34.29 73.66) (xy 68.58 73.66))
+    (stroke (width 0) (type default))
+  )
   (wire (pts (xy 200.66 55.88) (xy 204.47 55.88))
     (stroke (width 0) (type default))
@@
     (stroke (width 0) (type default))
   )
-  (wire (pts (xy 214.63 87.63) (xy 214.63 91.44))
+  (wire (pts (xy 214.63 81.28) (xy 214.63 91.44))
     (stroke (width 0) (type default))
   )
@@
     (stroke (width 0) (type default))
   )
-  (wire (pts (xy 34.29 73.66) (xy 68.58 73.66))
-    (stroke (width 0) (type default))
-  )
   (wire (pts (xy 88.9 153.67) (xy 88.9 157.48))
     (stroke (width 0) (type default))
@@
     (stroke (width 0) (type default))
   )
-  (wire (pts (xy 247.65 78.74) (xy 251.46 78.74))
+  (wire (pts (xy 247.65 78.74) (xy 255.27 78.74))
     (stroke (width 0) (type default))
   )
@@
     (stroke (width 0) (type default))
   )
-  (wire (pts (xy 68.58 73.66) (xy 68.58 39.37))
-    (stroke (width 0) (type default))
-  )
   (wire (pts (xy 172.72 20.32) (xy 175.26 20.32))
     (stroke (width 0) (type default))
   )
-  (wire (pts (xy 251.46 78.74) (xy 255.27 78.74))
-    (stroke (width 0) (type default))
-  )
   (wire (pts (xy 34.29 33.02) (xy 39.37 33.02))
     (stroke (width 0) (type default))
@@
     (stroke (width 0) (type default))
   )
-  (wire (pts (xy 214.63 87.63) (xy 251.46 87.63))
-    (stroke (width 0) (type default))
-  )
   (wire (pts (xy 46.99 92.71) (xy 60.96 92.71))
     (stroke (width 0) (type default))
@@
   )
   (wire (pts (xy 180.34 20.32) (xy 182.88 20.32))
+    (stroke (width 0) (type default))
+  )
+  (wire (pts (xy 68.58 39.37) (xy 68.58 73.66))
     (stroke (width 0) (type default))
   )
@@
     (effects (font (size 1.27 1.27)) (justify left bottom))
   )
+  (label "TWI_SDA" (at 162.56 92.71 90) (fields_autoplaced)
+    (effects (font (size 1.27 1.27)) (justify left bottom))
+  )
   (label "GPIO6" (at 39.37 43.18 0) (fields_autoplaced)
     (effects (font (size 1.27 1.27)) (justify left bottom))
@@
     (effects (font (size 1.27 1.27)) (justify left bottom))
   )
+  (label "TWI_SCK" (at 165.1 92.71 90) (fields_autoplaced)
+    (effects (font (size 1.27 1.27)) (justify left bottom))
+  )
   (label "GPIO33" (at 185.42 92.71 90) (fields_autoplaced)
     (effects (font (size 1.27 1.27)) (justify left bottom))
@@
     (effects (font (size 1.27 1.27)) (justify left bottom))
   )
-  (label "TWI_SDA" (at 160.02 92.71 90) (fields_autoplaced)
+  (label "GPIO14" (at 160.02 92.71 90) (fields_autoplaced)
     (effects (font (size 1.27 1.27)) (justify left bottom))
   )
@@
     (effects (font (size 1.27 1.27)) (justify left bottom))
   )
-  (label "TWI_SCK" (at 162.56 92.71 90) (fields_autoplaced)
-    (effects (font (size 1.27 1.27)) (justify left bottom))
-  )
   (label "GND" (at 175.26 25.4 90) (fields_autoplaced)
     (effects (font (size 1.27 1.27)) (justify left bottom))
@@
     (effects (font (size 1.27 1.27)) (justify left bottom))
   )
-  (label "RESET" (at 40.64 73.66 0) (fields_autoplaced)
+  (label "GPIO14" (at 40.64 73.66 0) (fields_autoplaced)
     (effects (font (size 1.27 1.27)) (justify left bottom))
   )
@@
     (effects (font (size 1.27 1.27)) (justify left bottom))
   )
-  (label "GPIO16" (at 165.1 92.71 90) (fields_autoplaced)
-    (effects (font (size 1.27 1.27)) (justify left bottom))
-  )

Commit message: new update
Changed lines of the file:
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@@
   (symbol (lib_id "Connector:Conn_01x10_Pin") (at 193.04 134.62 0) (mirror y) (unit 1)
     (in_bom yes) (on_board yes) (dnp no)
-    (property "Reference" "J1" (at 192.405 119.38 0)
+    (property "Reference" "J1" (at 193.04 118.11 0)
       (effects (font (size 1.27 1.27)))
     )
-    (property "Value" "Conn_01x10_Pin RIGHT" (at 191.77 121.92 0)
+    (property "Value" "Conn_01x10_Pin RIGHT" (at 191.77 120.65 0)
       (effects (font (size 1.27 1.27)))
     )

Commit message: new update
Parts:
- Q3: value Q_Dual_PMOS_S1G1D2S2G2D1 -> DMP3098LDM-7; footprint Package_TO_SOT_SMD:SOT-363_SC-70-6 -> DMP3098LDM-7:SOT95P285X140-6N
Connections:
- net VCC is gone; now on net +3V0: C17.1, J2.1 (Pin_1), Q3.6 (D)
Changed lines of the file:
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@@
     (effects (font (size 1.27 1.27)) (justify left bottom))
-  )
-  (symbol (lib_id "power:VCC") (at 161.29 175.26 0) (mirror x) (unit 1)
-    (in_bom yes) (on_board yes) (dnp no)
-    (property "Reference" "#PWR023" (at 161.29 171.45 0)
-      (effects (font (size 1.27 1.27)) hide)
-    )
-    (property "Value" "VCC" (at 161.29 179.07 0)
-      (effects (font (size 1.27 1.27)))
-    )
-    (property "Footprint" "" (at 161.29 175.26 0)
-      (effects (font (size 1.27 1.27)) hide)
-    )
-    (property "Datasheet" "" (at 161.29 175.26 0)
-      (effects (font (size 1.27 1.27)) hide)
-    )
-    (pin "1")
-    (instances
-      (project "SURF"
-        (path "/7d813604-5eab-4300-85c0-71d454ff6748"
-          (reference "#PWR023") (unit 1)
-        )
-      )
-    )
   )
   (symbol (lib_id "power:GND") (at 218.44 148.59 0) (mirror y) (unit 1)
@@
         (path "/7d813604-5eab-4300-85c0-71d454ff6748"
           (reference "R20") (unit 1)
+        )
+      )
+    )
+  )
+  (symbol (lib_id "power:+3V0") (at 217.17 121.92 0) (unit 1)
+    (in_bom yes) (on_board yes) (dnp no)
+    (property "Reference" "#PWR04" (at 217.17 125.73 0)
+      (effects (font (size 1.27 1.27)) hide)
+    )
+    (property "Value" "+3V0" (at 215.9 118.11 0)
+      (effects (font (size 1.27 1.27)) (justify left))
+    )
+    (property "Footprint" "" (at 217.17 121.92 0)
+      (effects (font (size 1.27 1.27)) hide)
+    )
+    (property "Datasheet" "" (at 217.17 121.92 0)
+      (effects (font (size 1.27 1.27)) hide)
+    )
+    (pin "1")
+    (instances
+      (project "SURF"
+        (path "/7d813604-5eab-4300-85c0-71d454ff6748"
+          (reference "#PWR04") (unit 1)
         )
       )
@@
     )
   )
+  (symbol (lib_id "power:+3V0") (at 161.29 175.26 180) (unit 1)
+    (in_bom yes) (on_board yes) (dnp no)
+    (property "Reference" "#PWR012" (at 161.29 171.45 0)
+      (effects (font (size 1.27 1.27)) hide)
+    )
+    (property "Value" "+3V0" (at 162.56 179.07 0)
+      (effects (font (size 1.27 1.27)) (justify left))
+    )
+    (property "Footprint" "" (at 161.29 175.26 0)
+      (effects (font (size 1.27 1.27)) hide)
+    )
+    (property "Datasheet" "" (at 161.29 175.26 0)
+      (effects (font (size 1.27 1.27)) hide)
+    )
+    (pin "1")
+    (instances
+      (project "SURF"
+        (path "/7d813604-5eab-4300-85c0-71d454ff6748"
+          (reference "#PWR012") (unit 1)
+        )
+      )
+    )
+  )
   (symbol (lib_id "power:+5V") (at 127 175.26 180) (unit 1)
     (in_bom yes) (on_board yes) (dnp no)
@@
     )
   )
+  (symbol (lib_id "power:+3V0") (at 15.24 125.73 0) (unit 1)
+    (in_bom yes) (on_board yes) (dnp no)
+    (property "Reference" "#PWR011" (at 15.24 129.54 0)
+      (effects (font (size 1.27 1.27)) hide)
+    )
+    (property "Value" "+3V0" (at 13.97 121.92 0)
+      (effects (font (size 1.27 1.27)) (justify left))
+    )
+    (property "Footprint" "" (at 15.24 125.73 0)
+      (effects (font (size 1.27 1.27)) hide)
+    )
+    (property "Datasheet" "" (at 15.24 125.73 0)
+      (effects (font (size 1.27 1.27)) hide)
+    )
+    (pin "1")
+    (instances
+      (project "SURF"
+        (path "/7d813604-5eab-4300-85c0-71d454ff6748"
+          (reference "#PWR011") (unit 1)
+        )
+      )
+    )
+  )
   (symbol (lib_id "Device:Q_Dual_PMOS_S1G1D2S2G2D1") (at 33.02 130.81 90) (unit 1)
     (in_bom yes) (on_board yes) (dnp no)
-    (property "Reference" "Q3" (at 33.02 123.19 90)
-      (effects (font (size 1.27 1.27)))
-    )
-    (property "Value" "Q_Dual_PMOS_S1G1D2S2G2D1" (at 33.02 118.11 90)
-      (effects (font (size 1.27 1.27)))
-    )
-    (property "Footprint" "Package_TO_SOT_SMD:SOT-363_SC-70-6" (at 33.02 129.54 0)
+    (property "Reference" "Q3" (at 33.02 124.46 90)
+      (effects (font (size 1.27 1.27)))
+    )
+    (property "Value" "DMP3098LDM-7" (at 33.02 118.11 90)
+      (effects (font (size 1.27 1.27)))
+    )
+    (property "Footprint" "DMP3098LDM-7:SOT95P285X140-6N" (at 33.02 129.54 0)
       (effects (font (size 1.27 1.27)) hide)
     )
@@
     )
   )
-  (symbol (lib_id "power:VCC") (at 15.24 125.73 0) (unit 1)
-    (in_bom yes) (on_board yes) (dnp no)
-    (property "Reference" "#PWR04" (at 15.24 129.54 0)
-      (effects (font (size 1.27 1.27)) hide)
-    )
-    (property "Value" "VCC" (at 15.24 121.92 0)
-      (effects (font (size 1.27 1.27)))
-    )
-    (property "Footprint" "" (at 15.24 125.73 0)
-      (effects (font (size 1.27 1.27)) hide)
-    )
-    (property "Datasheet" "" (at 15.24 125.73 0)
-      (effects (font (size 1.27 1.27)) hide)
-    )
-    (pin "1")
-    (instances
-      (project "SURF"
-        (path "/7d813604-5eab-4300-85c0-71d454ff6748"
-          (reference "#PWR04") (unit 1)
-        )
-      )
-    )
-  )
   (symbol (lib_id "Device:C") (at 78.74 149.86 0) (unit 1)
     (in_bom yes) (on_board yes) (dnp no)
@@
         )
       )
-    )
-  )
-  (symbol (lib_id "power:VCC") (at 217.17 121.92 0) (mirror y) (unit 1)
-    (in_bom yes) (on_board yes) (dnp no)
-    (property "Reference" "#PWR012" (at 217.17 125.73 0)
-      (effects (font (size 1.27 1.27)) hide)
-    )
-    (property "Value" "VCC" (at 217.17 118.11 0)
-      (effects (font (size 1.27 1.27)))
-    )
-    (property "Footprint" "" (at 217.17 121.92 0)
-      (effects (font (size 1.27 1.27)) hide)
-    )
-    (property "Datasheet" "" (at 217.17 121.92 0)
-      (effects (font (size 1.27 1.27)) hide)
-    )
-    (pin "1")
-    (instances
-      (project "SURF"
-        (path "/7d813604-5eab-4300-85c0-71d454ff6748"
-          (reference "#PWR012") (unit 1)
-        )
-      )

Commit message: new update
Parts:
- removed Q3: DMP3098LDM-7, DMP3098LDM-7:SOT95P285X140-6N, symbol Device:Q_Dual_PMOS_S1G1D2S2G2D1
- added Q1: BSS84PWH6327XTSA1, Package_TO_SOT_SMD:SOT-523, symbol Device:Q_PMOS_GSD
- CAM1: footprint OV2640:FPC-24 -> UPDATE_OV2640:ov2640-fcp_1
- J1, J2: footprint CONN_01X10_CRAZTFLIE:CONN_PINHEADERS_01X10_CRAZYFLIE -> UPDATE_CRAZYFLIE:CONN_PINHEADERS_01X10_CRAZYFLIE
Connections:
- net +3V0: now also Q1.3 (D)
- net CAM_VCC: now also Q1.2 (S)
- net at R24.1: now also Q1.1 (G)
Changed lines of the file:
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@@
     (effects (font (size 1.5 1.5) (thickness 0.3) bold) (justify left bottom))
   )
-  (text "POWER SUPPLY FOR LED" (at 124.46 144.78 0)
+  (text "POWER SUPPLY FOR LED" (at 124.46 138.43 0)
     (effects (font (size 1.5 1.5) (thickness 0.3) bold) (justify left bottom))
   )
@@
     )
   )
+  (symbol (lib_id "Device:Q_PMOS_GSD") (at 33.02 130.81 90) (unit 1)
+    (in_bom yes) (on_board yes) (dnp no)
+    (property "Reference" "Q1" (at 33.02 119.38 90)
+      (effects (font (size 1.27 1.27)))
+    )
+    (property "Value" "BSS84PWH6327XTSA1" (at 31.75 121.92 90)
+      (effects (font (size 1.27 1.27)))
+    )
+    (property "Footprint" "Package_TO_SOT_SMD:SOT-523" (at 30.48 125.73 0)
+      (effects (font (size 1.27 1.27)) hide)
+    )
+    (property "Datasheet" "~" (at 33.02 130.81 0)
+      (effects (font (size 1.27 1.27)) hide)
+    )
+    (pin "1")
+    (pin "2")
+    (pin "3")
+    (instances
+      (project "SURF"
+        (path "/7d813604-5eab-4300-85c0-71d454ff6748"
+          (reference "Q1") (unit 1)
+        )
+      )
+    )
+  )
   (symbol (lib_id "Device:R") (at 88.9 78.74 90) (unit 1)
     (in_bom yes) (on_board yes) (dnp no)
@@
       (effects (font (size 1.27 1.27)))
     )
-    (property "Footprint" "OV2640:FPC-24" (at 25.4 25.4 0)
+    (property "Footprint" "UPDATE_OV2640:ov2640-fcp_1" (at 25.4 25.4 0)
       (effects (font (size 1.27 1.27)) hide)
     )
@@
         (path "/7d813604-5eab-4300-85c0-71d454ff6748"
           (reference "#PWR011") (unit 1)
-        )
-      )
-    )
-  )
-  (symbol (lib_id "Device:Q_Dual_PMOS_S1G1D2S2G2D1") (at 33.02 130.81 90) (unit 1)
-    (in_bom yes) (on_board yes) (dnp no)
-    (property "Reference" "Q3" (at 33.02 124.46 90)
-      (effects (font (size 1.27 1.27)))
-    )
-    (property "Value" "DMP3098LDM-7" (at 33.02 118.11 90)
-      (effects (font (size 1.27 1.27)))
-    )
-    (property "Footprint" "DMP3098LDM-7:SOT95P285X140-6N" (at 33.02 129.54 0)
-      (effects (font (size 1.27 1.27)) hide)
-    )
-    (property "Datasheet" "~" (at 33.02 129.54 0)
-      (effects (font (size 1.27 1.27)) hide)
-    )
-    (pin "1")
-    (pin "2")
-    (pin "6")
-    (pin "3")
-    (pin "4")
-    (pin "5")
-    (instances
-      (project "SURF"
-        (path "/7d813604-5eab-4300-85c0-71d454ff6748"
-          (reference "Q3") (unit 1)
         )
       )
@@
       (effects (font (size 1.27 1.27)))
     )
-    (property "Footprint" "CONN_01X10_CRAZTFLIE:CONN_PINHEADERS_01X10_CRAZYFLIE" (at 231.14 134.62 0)
+    (property "Footprint" "UPDATE_CRAZYFLIE:CONN_PINHEADERS_01X10_CRAZYFLIE" (at 231.14 134.62 0)
       (effects (font (size 1.27 1.27)) hide)
     )
@@
       (effects (font (size 1.27 1.27)))
     )
-    (property "Footprint" "CONN_01X10_CRAZTFLIE:CONN_PINHEADERS_01X10_CRAZYFLIE" (at 193.04 134.62 0)
-      (effects (font (size 1.27 1.27)) hide)
-    )
+    (property "Footprint" "UPDATE_CRAZYFLIE:CONN_PINHEADERS_01X10_CRAZYFLIE" (at 193.04 134.62 0)
+      (effects (font (size 1.27 1.27)) hide)
+    )
