File: SURF.kicad_pcb (KiCad board)
At the start: 2 copper layers, 10 parts, among them Q1 BC338, Q2 BC338, Q4 BC338, U6 NCP164CSN300T1G, U7 XC6206PxxxMR, U8 XC6206PxxxMR

Commit message: new update
Parts:
- removed D4, D5, D6: 1.5KExxCA, Diode_THT:D_DO-201AE_P15.24mm_Horizontal
- removed D7: 1N914, Diode_THT:D_DO-35_SOD27_P7.62mm_Horizontal
- removed Q1, Q2, Q4: BC338, Package_TO_SOT_THT:TO-92_Inline
- removed U6: NCP164CSN300T1G, Package_TO_SOT_SMD:SOT-223-3_TabPin2
- removed U7, U8: XC6206PxxxMR, Package_TO_SOT_SMD:SOT-23-3
- added C1: 15pF, CAPACITOR15PF:CAPC1608X87N, F.Cu at (162.6, 88.2)
- added C15: 0.1uF, CAPACITOR0.1UF:CAPC1608X90N, F.Cu at (162.6, 95.0)
- added C17: 10uF, CAPACITOR10UF:CAPC2012X145N, B.Cu at (162.6, 77.0)
- added C18: 10uF, CAPACITOR10UF:CAPC2012X145N, B.Cu at (174.4, 73.7)
- added C19: 10uF, CAPACITOR10UF:CAPC2012X145N, B.Cu at (190.5, 76.2)
- added C2: 0.1uF, CAPACITOR0.1UF:CAPC1608X90N, F.Cu at (162.6, 80.6)
- added C20: 0.1uF, CAPACITOR0.1UF:CAPC1608X90N, B.Cu at (190.5, 86.4)
- added C21: 0.1uF, CAPACITOR0.1UF:CAPC1608X90N, B.Cu at (184.7, 78.7)
- added C22: 10uF, CAPACITOR10UF:CAPC2012X145N, B.Cu at (171.7, 76.2)
- added C3: 10uF, CAPACITOR10UF:CAPC2012X145N, B.Cu at (181.5, 86.2)
- added C4: 0.1uF/50V(1%), CAPACITOR0.1UF50V:CAPC3216X170N, B.Cu at (173.8, 88.9)
- added C5: 0.1uF/50V(1%), CAPACITOR0.1UF50V:CAPC3216X170N, B.Cu at (181.5, 88.9)
- added C6: 0.1uF, CAPACITOR0.1UF:CAPC1608X90N, F.Cu at (191.2, 73.7)
- added CAM1: OV2640 CONNECTOR, OV2640:FPC-24, F.Cu at (177.1, 73.7)
- added D1: LED, LED_SMD:LED_0603_1608Metric, F.Cu at (161.8, 73.7)
- added IC1: TPS7A0212PDBVR, TPS7A0212PDBVR:SOT95P280X145-5N, B.Cu at (186.7, 74.6)
- added IC2: TPS7A0228PDBVR, TPS7A0228PDBVR:SOT95P280X145-5N, B.Cu at (179.1, 74.6)
- added J1: Conn_01x10_Pin RIGHT, CONN_01X10_CRAZTFLIE:CONN_PINHEADERS_01X10_CRAZYFLIE, B.Cu at (183.8, 73.8)
- added J2: Conn_01x10_Pin LEFT, CONN_01X10_CRAZTFLIE:CONN_PINHEADERS_01X10_CRAZYFLIE, B.Cu at (161.8, 73.8)
- added J3: Conn_01x04, Connector_PinHeader_2.54mm:PinHeader_1x04_P2.54mm_Vertical, B.Cu at (179.3, 81.3)
- added Q3: Q_Dual_PMOS_S1G1D2S2G2D1, Package_TO_SOT_SMD:SOT-363_SC-70-6, B.Cu at (166.7, 76.2)
- added R1: 1K, Resistor_SMD:R_0402_1005Metric, F.Cu at (165.1, 73.7)
- added R18: 5.1K, Resistor_SMD:R_0402_1005Metric, F.Cu at (161.5, 76.7)
- added R19: 4.7K, Resistor_SMD:R_0402_1005Metric, F.Cu at (170.7, 83.8)
- added R20: 4.7K, Resistor_SMD:R_0402_1005Metric, F.Cu at (183.4, 81.3)
- added R21: 4.7K, Resistor_SMD:R_0402_1005Metric, F.Cu at (182.6, 83.8)
- added R23: 10K, Resistor_SMD:R_0402_1005Metric, B.Cu at (182.9, 81.3)
- added R24: 1K, Resistor_SMD:R_0402_1005Metric, B.Cu at (170.2, 73.7)
- added R3: 0, Resistor_SMD:R_0402_1005Metric, F.Cu at (191.0, 76.2)
- added R4: 499 R, Resistor_SMD:R_0402_1005Metric, B.Cu at (173.7, 86.2)
- added S2: TS20-42-25-WT-160-SMT-TR, NEW-SWITCH:TS204225WT160SMTTR, B.Cu at (172.1, 96.5)
- added S3: TS20-42-25-WT-160-SMT-TR, NEW-SWITCH:TS204225WT160SMTTR, B.Cu at (181.4, 96.3)
- added U1: ESP32-S2-MINI-2, new:ESP32-S2-MINI-2, F.Cu at (176.4, 101.2)
Other:
- board outline added: 33 x 30.5 mm

Commit message: new update
Parts:
- added R2: 0, Resistor_SMD:R_0402_1005Metric, B.Cu at (170.9, 95.1)
- C6, R3: moved to B.Cu
- moved C15 31.6 mm to (184.3, 72.0), turned to 180 degrees
- moved C6 24.0 mm to (169.7, 84.3), turned to 180 degrees
- moved R24 23.8 mm to (181.9, 94.3)
- moved C21 19.0 mm to (166.1, 75.5), turned to -90 degrees
- moved R3 18.2 mm to (174.8, 84.4)
- moved Q3 17.9 mm to (182.8, 83.9)
- moved C17 17.4 mm to (178.6, 83.9), turned to -90 degrees
- moved C1 14.3 mm to (165.3, 74.2), turned to -90 degrees
- moved C3 14.2 mm to (173.4, 97.8), turned to -90 degrees
- moved R19 14.0 mm to (178.5, 72.2), turned to 0 degrees
- moved IC1 12.1 mm to (174.7, 75.7)
- moved C4 12.0 mm to (178.9, 99.8)
- moved R21 11.6 mm to (190.2, 75.1), turned to 90 degrees
- moved RESET1 11.4 mm to (172.2, 89.6)
- moved R20 11.0 mm to (190.1, 72.6), turned to -90 degrees
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- renumbered S2 to BOOT1, S3 to RESET1
Connections:
- C1 pad 1: Net-(CAM1-PCLK) -> /GPIO7
- C15 pad 2: Net-(CAM1-RESET) -> /RESET
- C2 pad 1: +3V3 -> VCC
- C3 pad 1: GND -> +3V0
- C4 pad 1: +3V3 -> VCC
- C5 pad 1: +3V3 -> VCC
- CAM1 pad P$25: (no net) -> GND
- CAM1 pad P$26: (no net) -> GND
- CAM1 pad P10: (no net) -> GND
- CAM1 pad P11: (no net) -> /GPIO9
- CAM1 pad P12: (no net) -> /GPIO10
- CAM1 pad P13: (no net) -> /GPIO11
- CAM1 pad P14: (no net) -> DOVDD
- CAM1 pad P15: (no net) -> DVDD
- CAM1 pad P16: (no net) -> /GPIO12
- CAM1 pad P17: (no net) -> /PWDN
- CAM1 pad P18: (no net) -> /GPIO13
- CAM1 pad P19: (no net) -> /RESET
- CAM1 pad P20: (no net) -> /TWI_SCK
- CAM1 pad P21: (no net) -> AVDD
- CAM1 pad P22: (no net) -> /TWI_SDA
- CAM1 pad P23: (no net) -> GND
- CAM1 pad P3: (no net) -> /GPIO2
- CAM1 pad P4: (no net) -> /GPIO3
- CAM1 pad P5: (no net) -> /GPIO4
- CAM1 pad P6: (no net) -> /GPIO5
- CAM1 pad P7: (no net) -> /GPIO6
- CAM1 pad P8: (no net) -> /GPIO7
- CAM1 pad P9: (no net) -> /GPIO8
- J3 pad 3: Net-(J3-Pin_3) -> /TXD0
- Q3 pad 2: Net-(Q3A-G) -> unconnected-(Q3A-G-Pad2)
- R1 pad 1: Net-(CAM1-PWDN) -> /PWDN
- R19 pad 1: Net-(CAM1-RESET) -> /RESET
- R20 pad 1: Net-(CAM1-SIO_C) -> /TWI_SCK
- R21 pad 1: Net-(CAM1-SIO_D) -> /TWI_SDA
- R23 pad 1: VCC -> Net-(IC1-IN)
- R23 pad 2: Net-(Q3A-G) -> Net-(R23-Pad2)
- R24 pad 1: Net-(Q3A-G) -> Net-(R23-Pad2)
- RESET1 pad 3: GND -> Net-(RESET1-COM_1)
Routing:
- added copper zone on B.Cu, net GND

Commit message: new update
Parts:
- added R5: 10K, Resistor_SMD:R_0402_1005Metric, F.Cu at (171.3, 98.7)
- moved R23 1.72 mm to (185.2, 87.7)
- moved C6 1.23 mm to (170.9, 84.5)
- moved R24 0.68 mm to (181.2, 94.4)
- moved C5 0.55 mm to (178.9, 96.8)
- moved J2 0.53 mm to (161.8, 73.2)
- moved J1 0.48 mm to (183.8, 73.3)
Connections:
- C18 pad 1: Net-(IC1-IN) -> /CAM_VCC
- C2 pad 1: VCC -> /CAM_VCC
- C4 pad 1: VCC -> +3V0
- C5 pad 1: VCC -> +3V0
- CAM1 pad P$25: GND -> (no net)
- CAM1 pad P$26: GND -> (no net)
- CAM1 pad P10: GND -> (no net)
- CAM1 pad P11: /GPIO9 -> (no net)
- CAM1 pad P12: /GPIO10 -> (no net)
- CAM1 pad P13: /GPIO11 -> (no net)
- CAM1 pad P14: DOVDD -> (no net)
- CAM1 pad P15: DVDD -> (no net)
- CAM1 pad P16: /GPIO12 -> (no net)
- CAM1 pad P17: /PWDN -> (no net)
- CAM1 pad P18: /GPIO13 -> (no net)
- CAM1 pad P19: /RESET -> (no net)
- CAM1 pad P20: /TWI_SCK -> (no net)
- CAM1 pad P21: AVDD -> (no net)
- CAM1 pad P22: /TWI_SDA -> (no net)
- CAM1 pad P23: GND -> (no net)
- CAM1 pad P3: /GPIO2 -> (no net)
- CAM1 pad P4: /GPIO3 -> (no net)
- CAM1 pad P5: /GPIO4 -> (no net)
- CAM1 pad P6: /GPIO5 -> (no net)
- CAM1 pad P7: /GPIO6 -> (no net)
- CAM1 pad P8: /GPIO7 -> (no net)
- CAM1 pad P9: /GPIO8 -> (no net)
- IC1 pad 1: Net-(IC1-IN) -> /CAM_VCC
- IC1 pad 3: unconnected-(IC1-EN-Pad3) -> /CAM_VCC
- IC2 pad 1: Net-(IC1-IN) -> /CAM_VCC
- IC2 pad 3: unconnected-(IC2-EN-Pad3) -> /CAM_VCC
- J3 pad 3: /TXD0 -> Net-(J3-Pin_3)
- Q3 pad 1: Net-(IC1-IN) -> /CAM_VCC
- Q3 pad 2: unconnected-(Q3A-G-Pad2) -> Net-(Q3A-G)
- R24 pad 1: Net-(R23-Pad2) -> Net-(Q3A-G)
- RESET1 pad 2: /SW_EN -> GND
- RESET1 pad 3: Net-(RESET1-COM_1) -> GND
- U1 pad 3: VCC -> +3V0
- U1 pad 45: /EN -> GND

Commit message: new update
Parts:
- removed C3: 10uF, CAPACITOR10UF:CAPC2012X145N
- removed C6: 0.1uF, CAPACITOR0.1UF:CAPC1608X90N
- removed R2, R3: 0, Resistor_SMD:R_0402_1005Metric
- moved J2 0.47 mm to (161.6, 72.8)
- moved J1 0.38 mm to (183.8, 72.9)
- moved R23 0.19 mm to (185.2, 87.5)
Connections:
- C15 pad 2: /RESET -> /GPIO14
- R19 pad 1: /RESET -> /GPIO14
- R5 pad 1: GND -> /EN
- RESET1 pad 2: GND -> /EN
- U1 pad 18: /TWI_SDA -> /GPIO14
- U1 pad 19: /TWI_SCK -> /TWI_SDA
- U1 pad 20: /GPIO16 -> /TWI_SCK
- U1 pad 45: GND -> /EN

Commit message: new update
Parts:
- removed R23: 10K, Resistor_SMD:R_0402_1005Metric
- moved R5 14.2 mm to (170.6, 84.5), turned to 0 degrees
- moved C4 3.13 mm to (176.3, 98.0)
- moved C5 2.84 mm to (176.4, 95.5)
- moved R4 2.04 mm to (171.5, 94.3), turned to -90 degrees
- moved R19 1.64 mm to (180.1, 72.0)
- moved R24 1.23 mm to (181.1, 95.6)
- moved C18 0.85 mm to (179.3, 77.0)
- moved J1 0.54 mm to (184.0, 72.4)
- moved C2 0.53 mm to (168.3, 72.0), turned to 180 degrees
- moved J2 0.48 mm to (161.6, 72.3)
- moved R1 0.41 mm to (174.3, 72.1)
- moved R18 0.40 mm to (162.1, 77.2)
- moved IC1 0.32 mm to (174.4, 75.7)
- moved C15 0.29 mm to (184.6, 72.1)
- moved C17 0.22 mm to (178.4, 83.8)
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Connections:
- CAM1 pad P$25: (no net) -> GND
- CAM1 pad P$26: (no net) -> GND
- CAM1 pad P1: (no net) -> unnconnected
- CAM1 pad P10: (no net) -> GND
- CAM1 pad P11: (no net) -> /GPIO9
- CAM1 pad P12: (no net) -> /GPIO10
- CAM1 pad P13: (no net) -> /GPIO11
- CAM1 pad P14: (no net) -> /CAM_VCC
- CAM1 pad P15: (no net) -> +1V2
- CAM1 pad P16: (no net) -> /GPIO12
- CAM1 pad P17: (no net) -> /PWDN
- CAM1 pad P18: (no net) -> /GPIO13
- CAM1 pad P19: (no net) -> /GPIO14
- CAM1 pad P2: (no net) -> unnconnected
- CAM1 pad P20: (no net) -> /TWI_SCK
- CAM1 pad P21: (no net) -> +2V8
- CAM1 pad P22: (no net) -> /TWI_SDA
- CAM1 pad P23: (no net) -> GND
- CAM1 pad P24: (no net) -> unnconnected
- CAM1 pad P3: (no net) -> /GPIO2
- CAM1 pad P4: (no net) -> /GPIO3
- CAM1 pad P5: (no net) -> /GPIO4
- CAM1 pad P6: (no net) -> /GPIO5
- CAM1 pad P7: (no net) -> /GPIO6
- CAM1 pad P8: (no net) -> /GPIO7
- CAM1 pad P9: (no net) -> /GPIO8
Routing:
- net GND: track 0.00 -> 102.3 mm, vias 0 -> 38
- net /TWI_SCK: track 0.00 -> 76.6 mm, vias 0 -> 5
- net /GPIO14: track 0.00 -> 61.8 mm, vias 0 -> 2
- net /TWI_SDA: track 0.00 -> 54.0 mm, vias 0 -> 5
- net /GPIO7: track 0.00 -> 38.8 mm, vias 0 -> 2
- net /GPIO2: track 0.00 -> 36.8 mm, vias 0 -> 2
- net /GPIO3: track 0.00 -> 36.5 mm, vias 0 -> 2
- net /GPIO4: track 0.00 -> 36.0 mm, vias 0 -> 2
- net /GPIO6: track 0.00 -> 32.8 mm, vias 0 -> 4
- net /GPIO5: track 0.00 -> 32.8 mm, vias 0 -> 2
- net /GPIO8: track 0.00 -> 32.3 mm, vias 0 -> 2
- net /GPIO10: track 0.00 -> 31.1 mm
- net /EN: track 0.00 -> 29.9 mm, vias 0 -> 1
- net /GPIO11: track 0.00 -> 25.1 mm, vias 0 -> 2
- net /GPIO12: track 0.00 -> 25.0 mm, vias 0 -> 4
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Other:
- board size 33 x 30.5 mm -> 33.8 x 31 mm

Commit message: new update
Parts:
- Q3: value Q_Dual_PMOS_S1G1D2S2G2D1 -> DMP3098LDM-7; footprint Package_TO_SOT_SMD:SOT-363_SC-70-6 -> DMP3098LDM-7:SOT95P285X140-6N
- R5: moved to B.Cu
- moved R5 12.2 mm to (167.7, 96.4), turned to 90 degrees
- moved C20 4.05 mm to (190.2, 73.3), turned to 90 degrees
- moved C19 3.72 mm to (190.6, 77.2), turned to -90 degrees
- moved C2 1.13 mm to (169.5, 72.2)
- moved R18 1.12 mm to (162.5, 76.2), turned to 180 degrees
- moved R19 1.08 mm to (179.0, 72.0), turned to 180 degrees
- moved Q3 0.94 mm to (181.9, 83.7)
- moved C17 0.86 mm to (177.5, 83.7)
- moved C18 0.85 mm to (180.1, 76.6)
- moved R4 0.75 mm to (172.2, 94.3)
- moved J3 0.55 mm to (180.5, 79.8)
- moved IC1 0.36 mm to (174.2, 76.0)
- moved R1 0.30 mm to (174.2, 72.4)
- moved C15 0.29 mm to (184.3, 72.0)
- moved R24 0.16 mm to (180.9, 95.7)
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Connections:
- C17 pad 1: VCC -> +3V0
- J2 pad 1: VCC -> +3V0
- Q3 pad 6: VCC -> +3V0
Routing:
- net /TWI_SCK: track 76.6 -> 28.1 mm, vias 5 -> 3
- net /GPIO14: track 61.8 -> 21.3 mm, vias 2 -> 0
- net /CAM_VCC: track 23.7 -> 55.0 mm, vias 7 -> 6
- net /TWI_SDA: track 54.0 -> 24.9 mm, vias 5 -> 2
- net GND: track 102.3 -> 74.7 mm, vias 38 -> 48
- net /GPIO11: track 25.1 -> 43.5 mm
- net /EN: track 29.9 -> 14.1 mm, vias 1 -> 2
- net /GPIO9: track 24.4 -> 36.8 mm
- net /GPIO7: track 38.8 -> 48.6 mm, vias 2 -> 4
- net /GPIO10: track 31.1 -> 40.4 mm, vias 0 -> 2
- net +1V2: track 14.7 -> 22.5 mm, vias 2 -> 1
- net VCC: track 6.23 -> 0.00 mm, vias 3 -> 0
- net /GPIO18: track 14.8 -> 20.1 mm, vias 1 -> 2
- net +2V8: track 21.1 -> 16.8 mm
- net +3V0: track 18.5 -> 22.7 mm, vias 6 -> 8
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Other:
- board size 33.8 x 31 mm -> 33 x 30.7 mm
- copper layers 2 -> 4

Commit message: new update
Connections:
- J1 pad 1: /GPIO18 -> GND
- J1 pad 3: unconnected-(J1-Pin_3-Pad3) -> GND
- J1 pad 5: unconnected-(J1-Pin_5-Pad5) -> GND
- J1 pad 7: unconnected-(J1-Pin_7-Pad7) -> GND
- J1 pad 9: unconnected-(J1-Pin_9-Pad9) -> GND
- J2 pad 1: +3V0 -> GND
- J2 pad 3: unconnected-(J2-Pin_3-Pad3) -> GND
- J2 pad 5: unconnected-(J2-Pin_5-Pad5) -> GND
- J2 pad 7: unconnected-(J2-Pin_7-Pad7) -> GND
Routing:
- net /GPIO9: track 36.8 -> 37.8 mm
- net /GPIO2: track 39.4 -> 40.1 mm
- net /GPIO10: track 40.4 -> 40.9 mm, vias 2 -> 4
- net /GPIO18: track 20.1 -> 20.0 mm, vias 2 -> 1
- net /GPIO13: vias 3 -> 2

Commit message: new update
Parts:
- removed Q3: DMP3098LDM-7, DMP3098LDM-7:SOT95P285X140-6N
- added Q1: BSS84PWH6327XTSA1, Package_TO_SOT_SMD:SOT-523, B.Cu at (124.8, 57.9)
- CAM1: footprint OV2640:FPC-24 -> UPDATE_OV2640:ov2640-fcp_1
- J1, J2: footprint CONN_01X10_CRAZTFLIE:CONN_PINHEADERS_01X10_CRAZYFLIE -> UPDATE_CRAZYFLIE:CONN_PINHEADERS_01X10_CRAZYFLIE
- moved C19 56.1 mm to (137.8, 58.4), turned to 90 degrees
- moved C17 55.3 mm to (126.5, 62.4)
- moved IC2 54.2 mm to (134.2, 58.2)
- moved C20 52.7 mm to (139.6, 58.3)
- moved C18 52.7 mm to (129.1, 63.4), turned to -90 degrees
- moved R4 52.1 mm to (127.1, 68.2)
- moved R21 46.7 mm to (146.1, 60.0), turned to 0 degrees
- moved R20 46.5 mm to (146.2, 57.5), turned to 0 degrees
- moved BOOT1 45.4 mm to (136.6, 74.8)
- moved J1 45.2 mm to (141.4, 57.1)
- moved U1 45.1 mm to (134.2, 85.2)
- moved CAM1 44.9 mm to (134.5, 59.3)
- moved J2 44.8 mm to (119.4, 57.2)
- moved J3 44.3 mm to (138.1, 67.1)
- moved R18 44.2 mm to (121.4, 59.8)
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Connections:
- J1 pad 1: GND -> /GPIO18
- J1 pad 3: GND -> unconnected-(J1-Pin_3-Pad3)
- J1 pad 5: GND -> unconnected-(J1-Pin_5-Pad5)
- J1 pad 7: GND -> unconnected-(J1-Pin_7-Pad7)
- J1 pad 9: GND -> unconnected-(J1-Pin_9-Pad9)
- J2 pad 1: GND -> +3V0
- J2 pad 3: GND -> unconnected-(J2-Pin_3-Pad3)
- J2 pad 5: GND -> unconnected-(J2-Pin_5-Pad5)
- J2 pad 7: GND -> unconnected-(J2-Pin_7-Pad7)
Routing:
- net GND: track 75.0 -> 126.4 mm, vias 48 -> 59
- net /CAM_VCC: track 55.0 -> 29.0 mm, vias 6 -> 1
- net Net-(Q1-G): track 21.0 -> 44.6 mm
- net /GPIO13: track 17.6 -> 37.9 mm
- net /GPIO12: track 21.2 -> 40.8 mm
- net /GPIO2: track 40.1 -> 54.3 mm
- net /GPIO3: track 38.3 -> 51.4 mm
- net /GPIO14: track 21.2 -> 34.1 mm, vias 0 -> 2
- net /GPIO4: track 37.5 -> 49.1 mm
- net /GPIO5: track 36.7 -> 47.1 mm
- net Net-(J3-Pin_3): track 15.5 -> 6.59 mm
- net /TXD0: track 3.91 -> 12.2 mm
- net /GPIO6: track 35.9 -> 42.5 mm
- net /EN: track 14.1 -> 8.16 mm, vias 2 -> 1
- net +1V2: track 22.5 -> 16.8 mm, vias 1 -> 2
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